File: lna_sma_10x.kicad_sch (KiCad schematic)
At the start: 0 parts

Commit message: Initial schematic complete
  added New_Library with LT1722
  added schematic.pdf
Parts:
- added C1, C5: 10u, symbol Device:C
- added C2: 160p, symbol Device:C
- added C3, C4: 0.1, symbol Device:C
- added C6, C7: 0.1u, symbol Device:C
- added J1, J3: Conn_Coaxial, Connector_Coaxial:SMA_Amphenol_132289_EdgeMount, symbol Connector:Conn_Coaxial
- added J2: Power In, Connector_Molex:Molex_Nano-Fit_105309-xx03_1x03_P2.50mm_Vertical, symbol Connector_Generic:Conn_01x03
- added R1, R2: 10K, symbol Device:R_US
- added R3, R7: 50R, symbol Device:R_US
- added R4: 500R, symbol Device:R_US
- added R5: 4K5, symbol Device:R_US
- added R6: 100R, symbol Device:R_US
- added U1: LT1722xS8, Package_SO:SOIC-8_3.9x4.9mm_P1.27mm, symbol New_Library:LT1722xS8
- added U2: BUF602xD, Package_SO:SOIC-8_3.9x4.9mm_P1.27mm, symbol Amplifier_Buffer:BUF602xD
Connections:
- new net: J3.1 (In), R7.2
- new net: C2.2, R2.1, R3.1
- new net: R3.2, U1.3 (+in)
- new net: C2.1, J1.1 (In), R1.1
- new net: R6.2, U2.4 (IN)
- new net: R5.2, R7.1, U2.8
- new net: R4.2, R5.1, U1.2 (-in)
- new net: R6.1, U1.6 (Out)
- new net +5V: C5.2, C6.2, C7.2, J2.1 (Pin_1), U1.7 (V+), U2.1 (V+)
- new net -5V: C1.1, C3.1, C4.1, J2.3 (Pin_3), U1.4 (V-), U2.5 (V-)
- new net GND: C1.2, C3.2, C4.2, C5.1, C6.1, C7.1, J1.2 (Ext), J2.2 (Pin_2), J3.2 (Ext), R1.2, R2.2, R4.1
Other:
- note added: "Amp Specs Noise: 3.8 nV/sqrt(Hz) 1.2 pA/sqrt(Hz) 2.5 to 10 V supply 200 MHz GBW 3.7-4.5 mA supply current"
- note added: "Buffer Specs Noise: 4.8 nV/sqrt(Hz) 2.1 pA/sqrt(Hz) 3-12 V supply 6 mA supply current GBW os 1 GHz should ensure stability"
- note added: "DC blocking/LP filter and ground current return f_{c} = 100 kHz"
- note added: "Input-referred voltage noise: <= 100 uV RMS For 20 MHz bandwidth: V noise density <= 23 nV/sqrt(Hz) I noise density <= 450 pA/sqrt(Hz) with 50R source Implies: R <= 32K C >= 400f"
- note added: "Non-inverting gain: 1+R_{f}/R_{g} = 10"

Commit message: Schematic & BOM complete
Split feedback R into 2 in series to get standard values
Added power connector to library to have output power pins
Added part numbers, data sheets, footprints in BOM
Parts:
- added R7: 1k2, Resistor_SMD:R_1206_3216Metric_Pad1.30x1.75mm_HandSolder, symbol Device:R_US
- C1, C5: footprint (none) -> Capacitor_SMD:C_1206_3216Metric_Pad1.33x1.80mm_HandSolder; Mfr (none) -> Samsung; Mfr Part (none) -> CL31A106KAHNNNF
- C2: footprint (none) -> Capacitor_SMD:C_1206_3216Metric_Pad1.33x1.80mm_HandSolder; Mfr (none) -> Kyocera AVX; Mfr Part (none) -> 12065A161JAT2A; Tol/Type 5%/X5R -> 5%/C0G
- C3, C4: value 0.1 -> 0.1u; footprint (none) -> Capacitor_SMD:C_1206_3216Metric_Pad1.33x1.80mm_HandSolder; Mfr (none) -> Samsung; Mfr Part (none) -> CL31B104KBCNNND
- C6, C7: footprint (none) -> Capacitor_SMD:C_1206_3216Metric_Pad1.33x1.80mm_HandSolder; Mfr (none) -> Samsung; Mfr Part (none) -> CL31B104KBCNNND
- J1, J3: Mfr (none) -> Amphenol; Mfr Part (none) -> 132289
- J2: footprint Connector_Molex:Molex_Nano-Fit_105309-xx03_1x03_P2.50mm_Vertical -> Connector_Molex:Molex_Nano-Fit_105313-xx03_1x03_P2.50mm_Horizontal; symbol Connector_Generic:Conn_01x03 -> New_Library:Power-NanoFit-01x03; Mfr (none) -> Molex; Mfr Part (none) -> 105313-1303
- R1, R2: footprint (none) -> Resistor_SMD:R_1206_3216Metric_Pad1.30x1.75mm_HandSolder; Mfr (none) -> Vishay; Mfr Part (none) -> CRCW120610K0FKEBC; Tol/Type 5% -> 1%
- R3: footprint (none) -> Resistor_SMD:R_1206_3216Metric_Pad1.30x1.75mm_HandSolder; Mfr (none) -> Vishay; Mfr Part (none) -> CRCW120649R9FKEAC
- R4: footprint (none) -> Resistor_SMD:R_1206_3216Metric_Pad1.30x1.75mm_HandSolder; Mfr (none) -> Vishay; Mfr Part (none) -> CRCW1206499RFKEAC
- R5: value 4K5 -> 3K3; footprint (none) -> Resistor_SMD:R_1206_3216Metric_Pad1.30x1.75mm_HandSolder; Mfr (none) -> Vishay; Mfr Part (none) -> CRCW12063K32FKEAC
- R6: footprint (none) -> Resistor_SMD:R_1206_3216Metric_Pad1.30x1.75mm_HandSolder; Mfr (none) -> Vishay; Mfr Part (none) -> CRCW1206100RFKEAC
- R8: renamed from R7; footprint (none) -> Resistor_SMD:R_1206_3216Metric_Pad1.30x1.75mm_HandSolder; Mfr (none) -> Vishay; Mfr Part (none) -> CRCW120649R9FKEAC
- U1: Mfr (none) -> Analog Devices; Mfr Part (none) -> LT1722CS8#PBF
- U2: Mfr (none) -> Texas Instruments; Mfr Part (none) -> BUF602ID
Connections:
- net at R8.1, U2.8: now also R7.2; no longer R5.2
- new net: R5.2, R7.1
- no-connect marks 0 -> 1

Commit message: PCB Placement, setup for 4 layers
Connections:
- net sig_out: now reaches J3.1 (In), R8.2
- net R5toR7: now reaches R5.2, R7.1
- net buf_out: now reaches R7.2, R8.1, U2.8
- net sig_in_ac: now reaches C2.2, R2.1, R3.1
- net amp_in: now reaches R3.2, U1.3 (+in)
- net sig_in: now reaches C2.1, J1.1 (In), R1.1
- net buf_in: now reaches R6.2, U2.4 (IN)
- net fb_in: now reaches R4.2, R5.1, U1.2 (-in)
- net amp_out: now reaches R6.1, U1.6 (Out)
Changed lines of the file:
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@@
+    (effects (font (size 1.27 1.27)) (justify left bottom))
+  )
+  (label "buf_in" (at 140.97 92.71 0)
+    (effects (font (size 1.27 1.27)) (justify left bottom))
+  )
+  (label "sig_in" (at 29.21 96.52 0)
+    (effects (font (size 1.27 1.27)) (justify left bottom))
+  )
+  (label "sig_in_ac" (at 57.15 96.52 0)
+    (effects (font (size 1.27 1.27)) (justify left bottom))
+  )
+  (label "R5toR7" (at 139.7 71.12 0)
+    (effects (font (size 1.27 1.27)) (justify left bottom))
+  )
+  (label "buf_out" (at 162.56 71.12 0)
+    (effects (font (size 1.27 1.27)) (justify left bottom))
+  )
+  (label "amp_in" (at 78.74 96.52 0)
+    (effects (font (size 1.27 1.27)) (justify left bottom))
+  )
+  (label "sig_out" (at 189.23 92.71 0)
+    (effects (font (size 1.27 1.27)) (justify left bottom))
+  )
+  (label "amp_out" (at 113.03 92.71 0)
+    (effects (font (size 1.27 1.27)) (justify left bottom))
+  )
+  (label "fb_in" (at 100.33 71.12 0)
     (effects (font (size 1.27 1.27)) (justify left bottom))
   )

Commit message: now use git submodule kicad_hugonlib for libs
  moved power nano-fit over there and deleted New_Library
Parts:
- J2: symbol New_Library:Power-NanoFit-01x03 -> HugonLib:Power-NanoFit-01x03
- U1: symbol New_Library:LT1722xS8 -> HugonLib:LT1722xS8
Changed lines of the file:
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@@
     (pin "2")
   )
-  (symbol (lib_id "New_Library:Power-NanoFit-01x03") (at 76.2 162.56 270) (unit 1)
+  (symbol (lib_id "HugonLib:Power-NanoFit-01x03") (at 76.2 162.56 270) (unit 1)
     (in_bom yes) (on_board yes)
     (property "Reference" "J2" (id 0) (at 81.28 161.2899 90)
@@
       (effects (font (size 1.27 1.27)) (justify left))
     )
-    (property "Footprint" "Connector_Molex:Molex_Nano-Fit_105313-xx03_1x03_P2.50mm_Horizontal" (id 2) (at 76.2 162.56 0)
-      (effects (font (size 1.27 1.27)) hide)
-    )
-    (property "Datasheet" "https://www.mouser.com/datasheet/2/276/1/1053131303_PCB_HEADERS-1373923.pdf" (id 3) (at 76.2 162.56 0)
+    (property "Footprint" "Connector_Molex:Molex_Nano-Fit_105313-xx03_1x03_P2.50mm_Horizontal" (id 2) (at 83.82 162.56 0)
+      (effects (font (size 1.27 1.27)) hide)
+    )
+    (property "Datasheet" "~" (id 3) (at 76.2 162.56 0)
       (effects (font (size 1.27 1.27)) hide)
     )
@@
     (pin "1")
   )
-  (symbol (lib_id "New_Library:LT1722xS8") (at 97.79 92.71 0) (unit 1)
+  (symbol (lib_id "HugonLib:LT1722xS8") (at 97.79 92.71 0) (unit 1)
     (in_bom yes) (on_board yes)
     (property "Reference" "U1" (id 0) (at 101.6 85.09 0))
